Commit message: oscillation code implemented, but no convergence

File: rotors_simulator/rotors_description/urdf/licasa1.xacro (robot description, xacro)
@@ -260,5 +260,6 @@
     <axis xyz="1 0 0"/>
     <dynamics damping="0.0" friction="0.0"/>
-    <limit effort="6.0" lower="${-150/180*pi*0}" upper="${150/180*pi*0}" velocity="6"/>
+    <limit effort="6.0" lower="${-150/180*pi}" upper="${150/180*pi}" velocity="6"/>
+    <!-- <limit effort="6.0" lower="${-150/180*pi*0}" upper="${150/180*pi*0}" velocity="6"/> -->
   </joint>
   <link name="shoulder_link_x">
@@ -275,4 +276,5 @@
     <axis xyz="0 1 0"/>
     <dynamics damping="0.0" friction="0.0"/>
+    <!-- <limit effort="6.0" lower="${-150/180*pi}" upper="${150/180*pi}" velocity="6"/> -->
     <limit effort="6.0" lower="${-150/180*pi*0}" upper="${150/180*pi*0}" velocity="6"/>
   </joint>
@@ -589,6 +591,6 @@
       <inertia ixx="1e-03" ixy="0.0" ixz="0.0" iyy="1e-03" iyz="0.0" izz="1e-03"/>
     </inertial>
-  </link>
-  <joint name="left_eef_joint_1" type="revolute">
+  </link> -->
+  <!-- <joint name="left_eef_joint_1" type="revolute">
     <origin xyz="0 0 0"/>
     <parent link="left_eef_link"/>
@@ -605,5 +607,5 @@
     </inertial>
   </link>  -->
-  <gazebo>
+  <!-- <gazebo>
     <plugin name="f3d_plugin" filename="libgazebo_ros_f3d.so">
       <robotNamespace>licasa1</robotNamespace>
@@ -618,5 +620,5 @@
       <topicName>right_eef_link/body_wrench</topicName>
     </plugin>
-  </gazebo>
+  </gazebo> -->
   <!-- GRASP PLUGIN -->
   <!-- <gazebo>

Commit message: Switched to simple pendulum model; doesn't work

File: rotors_simulator/rotors_description/urdf/licasa1.xacro (robot description, xacro)
@@ -260,6 +260,6 @@
     <axis xyz="1 0 0"/>
     <dynamics damping="0.0" friction="0.0"/>
-    <limit effort="6.0" lower="${-150/180*pi}" upper="${150/180*pi}" velocity="6"/>
-    <!-- <limit effort="6.0" lower="${-150/180*pi*0}" upper="${150/180*pi*0}" velocity="6"/> -->
+    <!-- <limit effort="6.0" lower="${-150/180*pi}" upper="${150/180*pi}" velocity="6"/> -->
+    <limit effort="6.0" lower="${-150/180*pi*0}" upper="${150/180*pi*0}" velocity="6"/>
   </joint>
   <link name="shoulder_link_x">
