Commit message: adding damping

File: uav-cable-suspended-robots/uav-cable-suspended-robots-ros-pkg/urdf/licasa1_cube.urdf.xacro (robot description, xacro)
@@ -6,12 +6,12 @@
       <origin rpy="0 0 0" xyz="0 0 0"/>
       <mass value="0.25" />
-      <!-- <inertia ixx="1.5e-2" ixy="0.0" ixz="0.0" iyy="1.5e-2" iyz="0.0" izz="1.5e-2"/> mass 1 size 0.3 -->
+      <inertia ixx="0.375e-2" ixy="0.0" ixz="0.0" iyy="0.375e-2" iyz="0.0" izz="0.375e-2"/> <!-- mass 0.25 size 0.3 -->
       <!-- <inertia ixx="3e-3" ixy="0.0" ixz="0.0" iyy="2.167e-3" iyz="0.0" izz="2.167e-3"/> size 0.2 0.3 0.3-->
-      <inertia ixx="3.75e-3" ixy="0.0" ixz="0.0" iyy="2.083e-3" iyz="0.0" izz="2.083e-3"/>
+      <!-- <inertia ixx="3.75e-3" ixy="0.0" ixz="0.0" iyy="2.083e-3" iyz="0.0" izz="2.083e-3"/> mass 0.25 size 0.1 0.3 0.3 -->
     </inertial>
     <visual>
       <origin xyz="0 0 0"/>
       <geometry>
-	      <box size="0.1 0.3 0.3"/>
+	      <box size="0.3 0.3 0.3"/>
       </geometry>
     </visual>
@@ -19,5 +19,5 @@
       <origin xyz="0 0 0"/>
       <geometry>
-	      <box size="0.1 0.3 0.3"/>
+	      <box size="0.3 0.3 0.3"/>
       </geometry>
     </collision>
